File: GlacTracker7/tracker.brd (EAGLE design)
At the start: 160 x 89.3 mm, 79 parts, among them J1 THING_PLUS_PHYSICAL, J5 JST_6_PIN_VERTICAL, Q1 2N3906, Q2 AO6401A, Q3 DMN6070SY, U2 FONA-800-BREAKOUT, U3 MP2155GQ-Z, U4 SPARKFUN-SWARM-M138, U5 SPARKFUN-GPS-ZED-F9P, U6 MP2155GQ-Z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

Commit message: progress
Parts:
- removed J5: JST_6_PIN_VERTICAL, SparkFun-Connectors:JST-6-SMD-VERT-1.0MM
- removed JP4, JP5, JP6, JP7: (no value), jumper:JP2
- added C21: 1uF, resistor:C0805
- added JP8: (no value), jumper:JP1
- added Q6: MMBT3906LT1SMD, transistor-pnp:SOT23-BEC
- added Q7, Q8: DMG6602SVT, farnell-parts:TSOT26
- added R20, R21, R23: 100k, SparkFun-Resistors:0603
- added R22, R26: 100K, resistor:R0805
- added R24: 200R 0.1%, resistor:R0805
- added R25: 1K 0.1%, resistor:R0805
- added VCC_S: TPB2,54, testpad:B2,54
- Q2: value AO6401A -> DMG6602SVT; device GlacTracker:TSOP-6 -> farnell-parts:TSOT26
- Q3: value DMN6070SY -> DMG6602SVT; device GlacTracker:SOT-89-3 -> farnell-parts:TSOT26
- moved R19 179.2 mm to (60.2, 56.6), turned to 180 degrees
- moved R18 173.5 mm to (58.9, 50.0), turned to 90 degrees
- moved Q2 161.9 mm to (64.2, 51.1)
- moved Q3 130.6 mm to (33.5, 21.6), turned to 90 degrees
- moved Q1 88.7 mm to (48.5, 16.3)
- moved R1 83.0 mm to (58.2, 16.5), turned to 180 degrees
- moved R2 81.2 mm to (53.3, 14.0)
- moved U7 3.05 mm to (58.2, 23.1)
- moved U4 0.51 mm to (0.51, 0.00)
- moved U2 0.51 mm to (4.32, 44.5)
Connections:
- removed net GPS_RX1: J1.23, U5.13
- removed net GPS_TX1: J1.22, U5.14
- removed net GSM_EN: JP11.1, Q3.1, R19.1
- removed net GSM_PS: J1.9, U2.6
- removed net GSM_RX: J1.19, U2.10
- removed net GSM_TX: J1.4, U2.9
- removed net KEY: J1.8, U2.7
- removed net N$16: JP7.2, U6.6
- removed net N$4: JP5.2, U3.6
- removed net PSU_EN: J5.3, Q1.1, R2.2
- removed net SWARM_EN: J1.18, J5.1
- removed net SWARM_RX: J1.17, U4.5
- removed net SWARM_TX: J1.16, U4.7
- removed net VCC1_EN: J1.24, J5.2, JP7.1
- removed net VCC_1: TP6.P$1
- new net +3V3: Q7.P$2, R22.2
- new net ADC_7: C21.1, R24.2, R25.1
- new net BATV_EN: J1.23
- new net BATV_IN: J1.24
- new net COMMS_EN: J1.8, JP8.1, Q3.P$1, R21.1, U6.6, U6.7
- new net COMMS_RX: J1.9, U2.10, U4.5
- new net COMMS_TX: J1.4, U2.9, U4.7
- new net GNDA: C21.2, R24.1
- new net GPS_EN: J1.13, JP11.1, Q2.P$1, R19.1
- new net GSM_KEY: J1.3, U2.7
- new net N$35: Q3.P$3, Q3.P$6, R20.2
- new net SD_CS: J1.19
- new net SD_MISO: J1.16
- new net SD_MOSI: J1.17
- new net SD_SCK: J1.18
- new net SENSE_3V3: Q7.P$4, VCC_S.TP
- new net SENSE_EN: Q7.P$1, Q8.P$1
- new net SPARE: J1.20
- new net SPARE2: J1.21
- new net SPARE3: J1.22
- new net VCC: Q8.P$2, R26.2
- new net VCC_HP2_SW1: Q8.P$4, R25.2
- new net V_COMMS_IO: Q3.P$4, U2.12
- new net V_GPS: C1.1, C5.1, C7.1, Q2.P$4, U5.24, U5.3, U5.9, XB1.1
- net 3.3V: now also JP11.2, JP8.2, Q2.P$2, Q3.P$2, R18.1, R20.1; no longer C1.1, C5.1, C7.1, U2.12, U5.24, U5.3, U5.9, XB1.1
- net 3V3_EN: now also Q1.1, Q6.C, R2.2, R23.1, U3.6, U3.7; no longer JP5.1
- net 4.4V: now also C10.1, C3.1, C9.1, TP6.P$1, U2.1, U4.2
- net GND: now also Q2.P$5, Q3.P$5, Q7.P$5, Q8.P$5, R21.2, R23.2, U4.1; no longer JP4.1, JP6.1, Q3.3, U4.2
- net N$1: now also Q7.P$3, Q7.P$6, R22.1; no longer Q1.2, R1.2
- net N$12: now also Q8.P$3, Q8.P$6, R26.1; no longer JP6.2, U6.7
- net N$2: now also Q1.2, Q6.B, R1.2; no longer JP4.2, U3.7
- net N$34: now also Q2.P$3, Q2.P$6; no longer Q2.3, Q3.2, Q3.4
- net RTC_BAT: now also Q6.E
- net SCL: now also U5.15, U5.22
- net SDA: now also U5.12, U5.23
- net V_GSM: no longer C10.1, C9.1, Q2.1, Q2.2, Q2.5, Q2.6, U2.1
- net V_SWARM: no longer C3.1, U4.1
- net V_SYS: no longer JP11.2, JP4.3, JP5.3, JP6.3, JP7.3, Q2.4, R18.1
Routing:
- net 3.3V: track 16.2 -> 126.4 mm, vias 2 -> 4
- net SCL: track 0.00 -> 88.2 mm, vias 0 -> 1
- net SDA: track 0.00 -> 80.5 mm, vias 0 -> 1
- net V_GPS: track 0.00 -> 62.5 mm, vias 0 -> 1
- net COMMS_EN: track 0.00 -> 59.9 mm, vias 0 -> 3
- net COMMS_RX: track 0.00 -> 59.8 mm, vias 0 -> 2
- net RADIO_TX: track 0.00 -> 53.2 mm, vias 0 -> 1
- net RADIO_RX: track 0.00 -> 52.9 mm, vias 0 -> 1
- net COMMS_TX: track 0.00 -> 49.5 mm, vias 0 -> 1
- net GSM_RST: track 0.00 -> 34.4 mm, vias 0 -> 1
- net 4.4V: track 14.7 -> 47.4 mm
- net GSM_KEY: track 0.00 -> 29.3 mm, vias 0 -> 1
- net RTC_BAT: track 0.00 -> 29.1 mm
- net GPS_RX2: track 0.00 -> 26.3 mm
- net GPS_TX2: track 0.00 -> 26.2 mm
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Other:
- outline, holes or cut-outs redrawn

Commit message: Complete board for checking and naming
Parts:
- removed JP11, JP8: (no value), jumper:JP1
- removed LED1, LED2, LED3: (no value), led:CHIP-LED0805
- removed Q8: DMG6602SVT, farnell-parts:TSOT26
- removed R23: 100k, SparkFun-Resistors:0603
- removed R26: 100K, resistor:R0805
- removed TP5: TEST-POINTTP_15TH_THRU, SparkFun-Connectors:TP_15TH
- removed VCC_S: TPB2,54, testpad:B2,54
- added 3.3V, 4.4V, GPS, GSM: (no value), led:CHIP-LED0805
- added LED_EN: (no value), jumper:JP1
- added R27: 1k, SparkFun-Resistors:0603
- added U$1: ADAFRUIT-XTSD, GlacTracker:ADAFRUIT-XTSD
- JP1, JP2, JP3: value JUMPER-SMT_2_NC_TRACE_SILK -> (none); device SparkFun-Jumpers:SMT-JUMPER_2_NC_TRACE_SILK -> jumper:JP1
- R22: value 100K -> 100k; device resistor:R0805 -> SparkFun-Resistors:0603
- moved R24 196.8 mm to (117.1, 20.1)
- moved C21 196.3 mm to (117.1, 22.1), turned to 180 degrees
- moved R22 195.5 mm to (111.3, 17.0)
- moved R25 187.8 mm to (117.1, 16.8), turned to 180 degrees
- moved Q7 182.7 mm to (113.0, 20.8), turned to 270 degrees
- moved TP1 153.0 mm to (99.6, 10.2)
- moved C10 139.5 mm to (14.5, 36.1), turned to 0 degrees
- moved C9 131.9 mm to (25.9, 36.1), turned to 0 degrees
- moved JP2 129.7 mm to (28.3, 1.52), turned to 270 degrees
- moved TP3 129.4 mm to (70.9, 2.54)
- moved C3 121.3 mm to (4.39, 33.7), turned to 270 degrees
- moved C7 117.6 mm to (51.8, 85.2), turned to 270 degrees
- moved TP6 115.6 mm to (11.9, 1.27)
- moved C1 89.9 mm to (74.7, 63.8)
- moved C5 86.2 mm to (50.0, 85.2), turned to 270 degrees
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Connections:
- removed net +3V3: Q7.P$2, R22.2
- removed net ADC_7: C21.1, R24.2, R25.1
- removed net GNDA: C21.2, R24.1
- removed net N$1: Q7.P$3, Q7.P$6, R22.1
- removed net N$6: JP1.2, LED1.C
- removed net N$7: JP2.2, LED2.C
- removed net N$8: JP3.2, LED3.C
- removed net SENSE_3V3: Q7.P$4, VCC_S.TP
- removed net SENSE_EN: Q7.P$1, Q8.P$1
- removed net VCC: Q8.P$2, R26.2
- removed net VCC_2: TP5.P$1
- removed net V_GSM: R4.2
- removed net V_SWARM: R5.2
- new net N$3: 3.3V.C, 4.4V.C, GPS.C, GSM.C, LED_EN.2
- new net N$4: GPS.A, R4.1
- net 3.3V: now also JP2.2, JP3.2, U$1.3V3; no longer C6.1, C8.1, JP11.2, JP8.2
- net 3V3_EN: now also JP1.1; no longer R23.1
- net 4.4V: now also R5.2
- net BATV_EN: now also Q7.P$1
- net BATV_IN: now also C21.1, R24.2, R25.1
- net COMMS_EN: now also JP2.1; no longer JP8.1
- net GND: now also C21.2, J1.25, LED_EN.1, R24.1, U$1.GND; no longer JP1.1, JP2.1, JP3.1, Q8.P$5, R23.2
- net GPS_EN: now also JP3.1; no longer JP11.1
- net N$12: now also Q7.P$3, Q7.P$6, R22.2; no longer Q8.P$3, Q8.P$6, R26.1
- net N$13: now also 3.3V.A; no longer LED1.A
- net N$14: now also GSM.A, R27.1; no longer LED2.A, R4.1
- net N$15: now also 4.4V.A; no longer LED3.A
- net SD_CS: now also U$1.CS
- net SD_MISO: now also U$1.MISO
- net SD_MOSI: now also U$1.MOSI
- net SD_SCK: now also U$1.SCK
- net VCC_HP2_SW1: now also Q7.P$4; no longer Q8.P$4
- net V_BATT: now also Q7.P$2, R22.1
- net V_COMMS_IO: now also R27.2
- net V_GPS: now also C6.1, C8.1, R4.2
- net V_SYS: now also JP1.2
Routing:
- net 4.4V: track 47.4 -> 174.0 mm, vias 2 -> 4
- net V_GPS: track 62.5 -> 164.1 mm, vias 1 -> 4
- net V_COMMS_IO: track 22.8 -> 98.3 mm, vias 0 -> 2
- net 3.3V: track 126.4 -> 185.1 mm, vias 4 -> 7
- net BATV_IN: track 0.00 -> 58.0 mm, vias 0 -> 1
- net 3V3_EN: track 4.48 -> 59.2 mm, vias 0 -> 2
- net BATV_EN: track 0.00 -> 47.2 mm, vias 0 -> 2
- net SDA: track 80.5 -> 115.8 mm
- net SCL: track 88.2 -> 119.7 mm
- net COMMS_EN: track 59.9 -> 84.4 mm, vias 3 -> 5
- net SD_SCK: track 0.00 -> 19.1 mm
- net SD_MISO: track 0.00 -> 17.3 mm
- net N$3: track 0.00 -> 17.2 mm
- net V_SYS: track 94.7 -> 111.5 mm, vias 2 -> 6
- net SD_MOSI: track 0.00 -> 15.4 mm
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- added copper zone on layer 16, net GND
Other:
- board size 160 x 89.3 mm -> 120 x 89.3 mm
- board text added: "Headers: THING+ XTSD GPS RADIO GSM SWARM"
- board text added: "Misc: RTC 3V3_EN BATVOLTS_EN BATVOLTS_DIV"
- board text added: "Power: BAT CHG 3V3 V_GPS 4V4 V_GSMIO"
- board text removed: "3V3"
- board text removed: "PSU_EN"
- board text removed: "V_SWARM"

Commit message: added a break line
Routing:
- net GND: vias 192 -> 234
Other:
- outline, holes or cut-outs redrawn

Commit message: pre-tweak commt
Routing:
- net V_COMMS_IO: vias 2 -> 3
- net GSM_RST: vias 1 -> 2
- net GSM_KEY: vias 1 -> 2
- net GND: vias 234 -> 236
- net COMMS_TX: vias 1 -> 2
- net COMMS_RX: vias 2 -> 3
- net COMMS_EN: vias 5 -> 6
- net 4.4V: vias 4 -> 5
- net 3.3V: vias 7 -> 8
Other:
- board text added: "Graeme Bragg Kirk Martinez Sherif Attia ECS University of Southampton"
- board text added: "IT3"
- board text added: "V1.0"

Commit message: DRCand ERC run. Some tweaks to make to the Swarm/GSMoverlap
Connections:
- net COMMS_RX: now also J1.19; no longer J1.9
- net SD_CS: now also J1.20; no longer J1.19
- net SPARE: now also J1.9; no longer J1.20
Routing:
- net COMMS_RX: track 59.8 -> 75.4 mm, vias 3 -> 4
- net SD_CS: track 13.1 -> 16.3 mm, vias 1 -> 2
Changed lines of the file:
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@@
 <setting verticaltext="up"/>
 </settings>
-<grid distance="1" unitdist="mil" unit="mil" style="lines" multiple="1" display="yes" altdistance="5" altunitdist="mil" altunit="mil"/>
+<grid distance="10" unitdist="mil" unit="mil" style="lines" multiple="1" display="yes" altdistance="5" altunitdist="mil" altunit="mil"/>
 <layers>
 <layer number="1" name="Top" color="4" fill="1" visible="yes" active="yes"/>
@@
 <via x="49.53" y="27.559" extent="1-16" drill="0.4064" diameter="0.7112"/>
 <via x="49.53" y="25.019" extent="1-16" drill="0.4064" diameter="0.7112"/>
-<via x="49.53" y="40.259" extent="1-16" drill="0.4064" diameter="0.7112"/>
+<via x="49.5554" y="42.8498" extent="1-16" drill="0.4064" diameter="0.7112"/>
 <via x="49.53" y="45.339" extent="1-16" drill="0.4064" diameter="0.7112"/>
 <via x="50.546" y="51.689" extent="1-16" drill="0.4064" diameter="0.7112"/>
@@
 <contactref element="U4" pad="5"/>
 <wire x1="1.778" y1="43.18" x2="3.048" y2="44.45" width="0.3048" layer="16"/>
-<contactref element="J1" pad="9"/>
-<via x="46.101" y="42.164" extent="1-16" drill="0.3048"/>
-<wire x1="46.101" y1="42.164" x2="45.72" y2="42.545" width="0.3048" layer="16"/>
 <wire x1="45.72" y1="42.545" x2="43.561" y2="42.545" width="0.3048" layer="16"/>
 <via x="30.861" y="42.545" extent="1-16" drill="0.3048"/>
@@
 <wire x1="27.94" y1="44.45" x2="29.21" y2="45.72" width="0.3048" layer="16"/>
 <wire x1="29.21" y1="45.72" x2="29.21" y2="45.9994" width="0.3048" layer="16"/>
-<wire x1="48.006" y1="31.496" x2="46.482" y2="33.02" width="0.3048" layer="1"/>
-<wire x1="46.482" y1="33.02" x2="46.482" y2="41.783" width="0.3048" layer="1"/>
-<wire x1="46.482" y1="41.783" x2="46.101" y2="42.164" width="0.3048" layer="1"/>
 <wire x1="29.21" y1="45.9994" x2="29.972" y2="45.2374" width="0.3048" layer="1"/>
 <wire x1="29.972" y1="45.2374" x2="29.972" y2="43.434" width="0.3048" layer="1"/>
 <wire x1="29.972" y1="43.434" x2="30.861" y2="42.545" width="0.3048" layer="1"/>
 <via x="43.561" y="42.545" extent="1-16" drill="0.3048"/>
+<contactref element="J1" pad="19"/>
+<wire x1="68.326" y1="36.576" x2="64.516" y2="40.386" width="0.3048" layer="16"/>
+<wire x1="46.99" y1="40.386" x2="46.482" y2="40.894" width="0.3048" layer="16"/>
+<wire x1="46.482" y1="40.894" x2="46.482" y2="41.783" width="0.3048" layer="16"/>
+<wire x1="46.482" y1="41.783" x2="45.72" y2="42.545" width="0.3048" layer="16"/>
+<via x="46.99" y="40.386" extent="1-16" drill="0.3048"/>
+<wire x1="46.99" y1="40.386" x2="49.022" y2="40.386" width="0.254" layer="1"/>
+<via x="49.022" y="40.386" extent="1-16" drill="0.3048"/>
+<wire x1="49.022" y1="40.386" x2="46.99" y2="40.386" width="0.254" layer="16"/>
+<wire x1="64.516" y1="40.386" x2="49.022" y2="40.386" width="0.3048" layer="16"/>
 </signal>
 <signal name="COMMS_TX">
@@
 </signal>
 <signal name="SD_CS">
-<contactref element="J1" pad="19"/>
 <contactref element="U$1" pad="CS"/>
-<wire x1="68.326" y1="36.576" x2="70.231" y2="38.481" width="0.3048" layer="16"/>
-<wire x1="70.231" y1="38.481" x2="78.105" y2="38.481" width="0.3048" layer="16"/>
+<wire x1="70.231" y1="38.481" x2="70.4088" y2="38.481" width="0" layer="19" extent="1-16"/>
 <via x="78.105" y="38.481" extent="1-16" drill="0.3048"/>
+<wire x1="70.4088" y1="38.481" x2="78.105" y2="38.481" width="0.3048" layer="16"/>
 <wire x1="78.105" y1="38.481" x2="79.121" y2="39.497" width="0.3048" layer="1"/>
 <wire x1="79.121" y1="39.497" x2="79.121" y2="40.64" width="0.3048" layer="1"/>
+<contactref element="J1" pad="20"/>
+<wire x1="68.326" y1="34.036" x2="69.4944" y2="34.036" width="0.3048" layer="1"/>
+<wire x1="69.4944" y1="34.036" x2="69.9262" y2="34.4678" width="0.3048" layer="1"/>
+<wire x1="69.9262" y1="34.4678" x2="69.9262" y2="37.9984" width="0.3048" layer="1"/>
+<wire x1="69.9262" y1="37.9984" x2="70.4088" y2="38.481" width="0.3048" layer="1"/>
+<via x="70.4088" y="38.481" extent="1-16" drill="0.3048"/>
 </signal>
 <signal name="SD_MISO">
@@
 <via x="36.576" y="41.148" extent="1-16" drill="0.3048"/>
 <wire x1="36.576" y1="41.148" x2="37.338" y2="41.91" width="0.3048" layer="16"/>
-<wire x1="45.212" y1="41.91" x2="46.482" y2="40.64" width="0.3048" layer="16"/>
-<wire x1="46.482" y1="40.64" x2="46.482" y2="35.56" width="0.3048" layer="16"/>
-<wire x1="46.482" y1="35.56" x2="48.006" y2="34.036" width="0.3048" layer="16"/>
+<wire x1="45.212" y1="41.91" x2="45.974" y2="41.148" width="0.3048" layer="16"/>
+<wire x1="45.974" y1="41.148" x2="45.974" y2="36.068" width="0.3048" layer="16"/>
+<wire x1="45.974" y1="36.068" x2="48.006" y2="34.036" width="0.3048" layer="16"/>
 <wire x1="19.304" y1="17.526" x2="35.56" y2="17.526" width="0.3048" layer="16"/>
 <wire x1="28.702" y1="4.064" x2="28.702" y2="6.477" width="0.3048" layer="1"/>
@@
 <wire x1="110.744" y1="24.13" x2="110.236" y2="24.638" width="0.3048" layer="16"/>
 </signal>
-<signal name="SPARE">
-<contactref element="J1" pad="20"/>
-</signal>
 <signal name="SPARE2">
 <contactref element="J1" pad="21"/>
@@
 <wire x1="112.556" y1="37.338" x2="114.3" y2="37.338" width="0.3048" layer="1"/>
 </signal>
+<signal name="SPARE">
+<contactref element="J1" pad="9"/>
+</signal>
 </signals>

Commit message: missed and airwire
Parts:
- moved C25 0.25 mm to (100.1, 16.9)
- moved JP10 0.25 mm to (93.0, 20.1)
- moved JP2 0.25 mm to (28.3, 1.78)
Routing:
- net COMMS_RX: track 75.4 -> 77.1 mm

Commit message: track tweak
Routing:
- net COMMS_RX: track 77.1 -> 75.1 mm, vias 4 -> 2
Changed lines of the file:
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@@
 <setting verticaltext="up"/>
 </settings>
-<grid distance="10" unitdist="mil" unit="mil" style="lines" multiple="1" display="yes" altdistance="1" altunitdist="mil" altunit="mil"/>
+<grid distance="10" unitdist="mil" unit="mil" style="lines" multiple="1" display="yes" altdistance="5" altunitdist="mil" altunit="mil"/>
 <layers>
 <layer number="1" name="Top" color="4" fill="1" visible="yes" active="yes"/>
@@
 <via x="45.085" y="31.75" extent="1-16" drill="0.4064" diameter="0.7112"/>
 <via x="44.577" y="41.148" extent="1-16" drill="0.4064" diameter="0.7112"/>
-<via x="45.593" y="46.609" extent="1-16" drill="0.4064" diameter="0.7112"/>
+<via x="46.482" y="48.006" extent="1-16" drill="0.4064" diameter="0.7112"/>
 <via x="45.085" y="29.21" extent="1-16" drill="0.4064" diameter="0.7112"/>
 <via x="35.56" y="41.275" extent="1-16" drill="0.4064" diameter="0.7112"/>
@@
 <contactref element="U4" pad="5"/>
 <wire x1="1.778" y1="43.18" x2="3.048" y2="44.45" width="0.3048" layer="16"/>
-<wire x1="45.72" y1="42.545" x2="43.561" y2="42.545" width="0.3048" layer="16"/>
+<wire x1="46.101" y1="42.545" x2="43.561" y2="42.545" width="0.3048" layer="16"/>
 <via x="30.861" y="42.545" extent="1-16" drill="0.3048"/>
 <wire x1="43.561" y1="42.545" x2="30.861" y2="42.545" width="0.3048" layer="16"/>
@@
 <via x="43.561" y="42.545" extent="1-16" drill="0.3048"/>
 <contactref element="J1" pad="19"/>
-<wire x1="46.99" y1="40.386" x2="46.482" y2="40.894" width="0.3048" layer="16"/>
-<wire x1="46.482" y1="40.894" x2="46.482" y2="41.783" width="0.3048" layer="16"/>
-<wire x1="46.482" y1="41.783" x2="45.72" y2="42.545" width="0.3048" layer="16"/>
-<via x="46.99" y="40.386" extent="1-16" drill="0.3048"/>
-<wire x1="46.99" y1="40.386" x2="49.022" y2="40.386" width="0.254" layer="1"/>
-<via x="49.022" y="40.386" extent="1-16" drill="0.3048"/>
-<wire x1="49.022" y1="40.386" x2="46.99" y2="40.386" width="0.254" layer="16"/>
+<wire x1="47.244" y1="40.386" x2="46.736" y2="40.894" width="0.3048" layer="16"/>
+<wire x1="46.736" y1="40.894" x2="46.736" y2="41.91" width="0.3048" layer="16"/>
+<wire x1="46.736" y1="41.91" x2="46.101" y2="42.545" width="0.3048" layer="16"/>
+<wire x1="49.022" y1="40.386" x2="47.244" y2="40.386" width="0.3048" layer="16"/>
 <wire x1="68.326" y1="36.576" x2="67.056" y2="36.576" width="0.3048" layer="16"/>
 <wire x1="67.056" y1="36.576" x2="66.294" y2="37.338" width="0.3048" layer="16"/>
@@
 <via x="35.56" y="17.526" extent="1-16" drill="0.4064"/>
 <contactref element="J1" pad="8"/>
-<wire x1="45.212" y1="41.91" x2="43.942" y2="41.91" width="0.3048" layer="16"/>
+<wire x1="45.593" y1="41.91" x2="43.942" y2="41.91" width="0.3048" layer="16"/>
 <wire x1="43.942" y1="41.91" x2="37.338" y2="41.91" width="0.3048" layer="16"/>
 <wire x1="35.56" y1="19.45" x2="36.087" y2="19.45" width="0.3048" layer="1"/>
@@
 <via x="36.576" y="41.148" extent="1-16" drill="0.3048"/>
 <wire x1="36.576" y1="41.148" x2="37.338" y2="41.91" width="0.3048" layer="16"/>
-<wire x1="45.212" y1="41.91" x2="45.974" y2="41.148" width="0.3048" layer="16"/>
-<wire x1="45.974" y1="41.148" x2="45.974" y2="36.068" width="0.3048" layer="16"/>
-<wire x1="45.974" y1="36.068" x2="48.006" y2="34.036" width="0.3048" layer="16"/>
+<wire x1="45.593" y1="41.91" x2="46.101" y2="41.402" width="0.3048" layer="16"/>
+<wire x1="46.101" y1="41.402" x2="46.101" y2="35.941" width="0.3048" layer="16"/>
+<wire x1="46.101" y1="35.941" x2="48.006" y2="34.036" width="0.3048" layer="16"/>
 <wire x1="19.304" y1="17.526" x2="35.56" y2="17.526" width="0.3048" layer="16"/>
 <wire x1="28.702" y1="4.064" x2="28.702" y2="6.477" width="0.3048" layer="1"/>
